File: elec/layout/default/power-prioritiser.kicad_pcb (KiCad board)
At the start: 2 copper layers, 40 x 40 mm, 0 parts

Commit message: Initial content
Parts:
- added DS1: ?, lib:SOD-323_L1.8-W1.3-LS2.5-RD, F.Cu at (125.6, 88.9)
- added Q1: ?, lib:SOT-23_L2.9-W1.3-P1.90-LS2.4-BR, F.Cu at (125.6, 91.7)
- added R1: 100mW Thick Film Resistors 75V ±100ppm/℃ ±1% 10kΩ 0603 Chip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, lib:R0603, F.Cu at (128.0, 91.2)
Routing:
- net vcc: track 0.00 -> 3.32 mm
- net vcc-2: track 0.00 -> 1.76 mm
Other:
- board outline removed
- board text removed: "{{GITHASH}}"
